File: whylight.kicad_pcb (KiCad board)
At the start: 4 copper layers, 107.9 x 40 mm, 109 parts, among them J1 USB device, J2 External 5v, J3 External 5v, J4 I2C, J5 UART, J7 Ledstrip, U1 AG5405, U10 INA233, U11 L78L05_SOT89, U12 GM3085N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

Commit message: r0.1
Parts:
- added N1: Logo, library:logo_nicolai, B.Cu at (69.2, -15.0)
- moved C9 22.8 mm to (29.9, -14.5), turned to 90 degrees
- moved D10 2.25 mm to (24.1, -14.3)
Routing:
- net +VIN: track 182.2 -> 141.5 mm
- net GND: track 98.0 -> 132.3 mm, vias 81 -> 114
- net USB_P: track 63.4 -> 58.0 mm
- net USB_N: track 61.3 -> 55.9 mm
- net ETH_LED2A: track 56.5 -> 53.5 mm, vias 3 -> 2
- net Net-(D1-K): track 51.9 -> 50.7 mm
Other:
- board text added: "CLK"
- board text added: "DAT"
- board text added: "GND"
- board text added: "PWR"
- board text added: "© 2024 Nicolai Electronics CERN-OHL-P r0.1"
- board text removed: "- c d +"
- board text removed: "PoE+"
- board text removed: "© 2024 Nicolai Electronics CERN-OHL-P"

Commit message: Release r0.1
Parts:
- removed RJ1: HR913180AE, library:RJ45-TH_HR913180AE
- added J6: 0826-1X1T-GJ-F, library:BEL_0826-1X1T-GJ-F, F.Cu at (10.5, 0.00)
- added JP3: LDO_B, Jumper:SolderJumper-2_P1.3mm_Open_RoundedPad1.0x1.5mm, F.Cu at (87.4, -4.27)
- added JP4: LED power bypass, Jumper:SolderJumper-2_P1.3mm_Open_RoundedPad1.0x1.5mm, F.Cu at (87.4, -1.68)
- added JP5: LDO_E, Jumper:SolderJumper-2_P1.3mm_Open_RoundedPad1.0x1.5mm, F.Cu at (84.0, -1.68)
- moved D9 7.07 mm to (35.9, -12.4)
Connections:
- U11 pad 3: +VIN -> Net-(JP5-B)
Routing:
- net +5V: track 92.2 -> 101.4 mm
- net Net-(JP5-B): track 0.00 -> 4.00 mm
- net Net-(D1-K): track 50.7 -> 48.1 mm
- net +5v-USB: track 95.8 -> 98.1 mm
- net Net-(J6-Pad17): track 2.69 -> 3.68 mm
- net +VIN: track 141.5 -> 140.8 mm
- net Net-(D2-A): vias 8 -> 5
- net GND: vias 114 -> 119
