File: whylight.kicad_sch (KiCad schematic)
At the start: 80 parts, among them J1 USB device, J2 External 5v, J3 External 5v, J4 I2C, J5 UART, J7 Ledstrip, U1 AG5405, U10 INA233, U11 L78L05_SOT89, U12 GM3085N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

Commit message: Release r0.1
Parts:
- added JP3: LDO_B, Jumper:SolderJumper-2_P1.3mm_Open_RoundedPad1.0x1.5mm, symbol Jumper:Jumper_2_Open
- added JP4: LED power bypass, Jumper:SolderJumper-2_P1.3mm_Open_RoundedPad1.0x1.5mm, symbol Jumper:Jumper_2_Open
- added JP5: LDO_E, Jumper:SolderJumper-2_P1.3mm_Open_RoundedPad1.0x1.5mm, symbol Jumper:Jumper_2_Open
- L1: LCSC C7427114 -> C167928
- R23, R5: LCSC C2935237 -> C11702
Connections:
- net +5V: now also JP3.2 (B)
- net +5v-USB: now also JP4.1 (A)
- net +VIN: now also JP3.1 (A), JP4.2 (B), JP5.1 (A); no longer U11.3 (IN)
- new net: JP5.2 (B), U11.3 (IN)
Other:
- moved on the sheet: C21, JP2, U11
